Commit message: Configured Arm for Pickup

File: amr_ws/src/robot_arm_description/urdf/urdf_backup.xacro (robot description, xacro)
@@ -111,5 +111,12 @@
             <material name="silver" />
         </visual>
-        </link>
+        <collision>
+            <origin xyz="0.000154 3.6e-05 -0.075138" rpy="0 0 0" />
+            <geometry>
+                <mesh filename="file://$(find robot_arm_description)/meshes/Bearing_clamp_1.stl"
+                    scale="0.001 0.001 0.001" />
+            </geometry>
+        </collision>
+    </link>
     <link name="Bearing_ring_1">
         <inertial>
@@ -127,5 +134,12 @@
             <material name="silver" />
         </visual>
-        </link>
+        <collision>
+            <origin xyz="0.000156 3.6e-05 -0.078638" rpy="0 0 0" />
+            <geometry>
+                <mesh filename="file://$(find robot_arm_description)/meshes/Bearing_ring_1.stl"
+                    scale="0.001 0.001 0.001" />
+            </geometry>
+        </collision>
+    </link>
     <link name="Gear_12T_1">
         <inertial>
@@ -143,5 +157,12 @@
             <material name="silver" />
         </visual>
-        </link>
+        <collision>
+            <origin xyz="0.048113 -0.009181 -0.075108" rpy="0 0 0" />
+            <geometry>
+                <mesh filename="file://$(find robot_arm_description)/meshes/Gear_12T_1.stl"
+                    scale="0.001 0.001 0.001" />
+            </geometry>
+        </collision>
+    </link>
     <link name="Gear_27T_1">
         <inertial>
@@ -159,5 +180,12 @@
             <material name="silver" />
         </visual>
-        </link>
+        <collision>
+            <origin xyz="-0.040402 -0.012281 -0.075166" rpy="0 0 0" />
+            <geometry>
+                <mesh filename="file://$(find robot_arm_description)/meshes/Gear_27T_1.stl"
+                    scale="0.001 0.001 0.001" />
+            </geometry>
+        </collision>
+    </link>
     <link name="Potentiometer_1">
         <inertial>
@@ -175,5 +203,12 @@
             <material name="silver" />
         </visual>
-        </link>
+        <collision>
+            <origin xyz="0.04815 -0.000182 -0.070107" rpy="0 0 0" />
+            <geometry>
+                <mesh filename="file://$(find robot_arm_description)/meshes/Potentiometer_1.stl"
+                    scale="0.001 0.001 0.001" />
+            </geometry>
+        </collision>
+    </link>
     <link name="Steel_ball_10mm_1">
         <inertial>
@@ -191,5 +226,11 @@
             <material name="silver" />
         </visual>
-        </link>
+        <collision>
+            <origin xyz="-0.055442 -0.039976 -0.079735" rpy="0 0 0" />
+            <geometry>
+                <sphere radius="0.005" />
+            </geometry>
+        </collision>
+    </link>
     <link name="Steel_ball_10mm_4">
         <inertial>
@@ -207,5 +248,11 @@
             <material name="silver" />
         </visual>
-        </link>
+        <collision>
+            <origin xyz="-0.021305 -0.065014 -0.079717" rpy="0 0 0" />
+            <geometry>
+                <sphere radius="0.005" />
+            </geometry>
+        </collision>
+    </link>
     <link name="Steel_ball_10mm_3">
         <inertial>
@@ -223,5 +270,11 @@
             <material name="silver" />
         </visual>
-        </link>
+        <collision>
+            <origin xyz="0.02103 -0.065206 -0.07969" rpy="0 0 0" />
+            <geometry>
+                <sphere radius="0.005" />
+            </geometry>
+        </collision>
+    </link>
     <link name="Steel_ball_10mm_2">
         <inertial>
@@ -239,5 +292,11 @@
             <material name="silver" />
         </visual>
-        </link>
+        <collision>
+            <origin xyz="0.055392 -0.040477 -0.079664" rpy="0 0 0" />
+            <geometry>
+                <sphere radius="0.005" />
+            </geometry>
+        </collision>
+    </link>
     <link name="Steel_ball_10mm_10">
         <inertial>
@@ -255,5 +314,11 @@
             <material name="silver" />
         </visual>
-        </link>
+        <collision>
+            <origin xyz="0.068656 -0.000273 -0.079648" rpy="0 0 0" />
+            <geometry>
+                <sphere radius="0.005" />
+            </geometry>
+        </collision>
+    </link>
     <link name="Steel_ball_10mm_9">
         <inertial>
@@ -271,5 +336,11 @@
             <material name="silver" />
         </visual>
-        </link>
+        <collision>
+            <origin xyz="-0.068342 0.000346 -0.079736" rpy="0 0 0" />
+            <geometry>
+                <sphere radius="0.005" />
+            </geometry>
+        </collision>
+    </link>
     <link name="Steel_ball_10mm_8">
         <inertial>
@@ -287,5 +358,11 @@
             <material name="silver" />
         </visual>
-        </link>
+        <collision>
+            <origin xyz="-0.055078 0.04055 -0.079721" rpy="0 0 0" />
+            <geometry>
+                <sphere radius="0.005" />
+            </geometry>
+        </collision>
+    </link>
     <link name="Steel_ball_10mm_5">
         <inertial>
@@ -303,5 +380,11 @@
             <material name="silver" />
         </visual>
-        </link>
+        <collision>
+            <origin xyz="-0.020716 0.065279 -0.079695" rpy="0 0 0" />
+            <geometry>
+                <sphere radius="0.005" />
+            </geometry>
+        </collision>
+    </link>
     <link name="Steel_ball_10mm_6">
         <inertial>
@@ -319,5 +402,11 @@
             <material name="silver" />
         </visual>
-        </link>
+        <collision>
+            <origin xyz="0.021619 0.065088 -0.079668" rpy="0 0 0" />
+            <geometry>
+                <sphere radius="0.005" />
+            </geometry>
+        </collision>
+    </link>
     <link name="Steel_ball_10mm_7">
         <inertial>
@@ -335,5 +424,11 @@
             <material name="silver" />
         </visual>
-        </link>
+        <collision>
+            <origin xyz="0.055756 0.040049 -0.07965" rpy="0 0 0" />
+            <geometry>
+                <sphere radius="0.005" />
+            </geometry>
+        </collision>
+    </link>
     <link name="Bearing_clamp_2">
         <inertial>
@@ -351,5 +446,12 @@
             <material name="silver" />
         </visual>
-        </link>
+        <collision>
+            <origin xyz="0.000112 2.5e-05 -0.010138" rpy="0 0 0" />
+            <geometry>
+                <mesh filename="file://$(find robot_arm_description)/meshes/Bearing_clamp_2.stl"
+                    scale="0.001 0.001 0.001" />
+            </geometry>
+        </collision>
+    </link>
     <link name="Rotating_plate_1">
         <inertial>
@@ -391,5 +493,13 @@
             <material name="silver" />
         </visual>
-        </link>
+        <collision>
+            <origin xyz="0.000114 2.6e-05 -0.013192" rpy="0 0 0" />
+            <geometry>
+                <mesh
+                    filename="file://$(find robot_arm_description)/meshes/Rotating_plate_clamp_1.stl"
+                    scale="0.001 0.001 0.001" />
+            </geometry>
+        </collision>
+    </link>
     <link name="Base_servo_mount_1">
         <inertial>
@@ -501,5 +611,13 @@
             <material name="silver" />
         </visual>
-        </link>
+        <collision>
+            <origin xyz="0.01774 -0.120366 -0.145201" rpy="0 0 0" />
+            <geometry>
+                <mesh
+                    filename="file://$(find robot_arm_description)/meshes/Lower_arm_bushing__1__1.stl"
+                    scale="0.001 0.001 0.001" />
+            </geometry>
+        </collision>
+    </link>
     <link name="Lower_arm_bushing_1">
         <inertial>
@@ -517,5 +635,12 @@
             <material name="silver" />
         </visual>
-        </link>
+        <collision>
+            <origin xyz="0.018133 -0.065367 -0.145192" rpy="0 0 0" />
+            <geometry>
+                <mesh filename="file://$(find robot_arm_description)/meshes/Lower_arm_bushing_1.stl"
+                    scale="0.001 0.001 0.001" />
+            </geometry>
+        </collision>
+    </link>
     <link name="Center_arm_1">
         <inertial>
@@ -556,5 +681,13 @@
             <material name="silver" />
         </visual>
-        </link>
+        <collision>
+            <origin xyz="-0.010723 -0.185164 -0.14523" rpy="0 0 0" />
+            <geometry>
+                <mesh
+                    filename="file://$(find robot_arm_description)/meshes/Center_arm_bearing_guide__1__1.stl"
+                    scale="0.001 0.001 0.001" />
+            </geometry>
+        </collision>
+    </link>
     <link name="Bearing_holder_1">
         <inertial>
@@ -572,5 +705,12 @@
             <material name="silver" />
         </visual>
-        </link>
+        <collision>
+            <origin xyz="-0.024123 -0.185068 -0.145239" rpy="0 0 0" />
+            <geometry>
+                <mesh filename="file://$(find robot_arm_description)/meshes/Bearing_holder_1.stl"
+                    scale="0.001 0.001 0.001" />
+            </geometry>
+        </collision>
+    </link>
     <link name="Center_arm_bearing_guide_1">
         <inertial>
@@ -589,5 +729,13 @@
             <material name="silver" />
         </visual>
-        </link>
+        <collision>
+            <origin xyz="-0.010648 -0.185145 -0.26273" rpy="0 0 0" />
+            <geometry>
+                <mesh
+                    filename="file://$(find robot_arm_description)/meshes/Center_arm_bearing_guide_1.stl"
+                    scale="0.001 0.001 0.001" />
+            </geometry>
+        </collision>
+    </link>
     <link name="Bearing_holder__1__1">
         <inertial>
@@ -606,5 +754,13 @@
             <material name="silver" />
         </visual>
-        </link>
+        <collision>
+            <origin xyz="-0.024047 -0.185049 -0.262739" rpy="0 0 0" />
+            <geometry>
+                <mesh
+                    filename="file://$(find robot_arm_description)/meshes/Bearing_holder__1__1.stl"
+                    scale="0.001 0.001 0.001" />
+            </geometry>
+        </collision>
+    </link>
     <link name="Center_arm_bearing_guide_clamp__1__1">
         <inertial>
@@ -623,5 +779,13 @@
             <material name="silver" />
         </visual>
-        </link>
+        <collision>
+            <origin xyz="-0.032523 -0.185008 -0.145244" rpy="0 0 0" />
+            <geometry>
+                <mesh
+                    filename="file://$(find robot_arm_description)/meshes/Center_arm_bearing_guide_clamp__1__1.stl"
+                    scale="0.001 0.001 0.001" />
+            </geometry>
+        </collision>
+    </link>
     <link name="Center_arm_bearing_guide_clamp__2__1">
         <inertial>
@@ -640,5 +804,13 @@
             <material name="silver" />
         </visual>
-        </link>
+        <collision>
+            <origin xyz="-0.024047 -0.185049 -0.262739" rpy="0 0 0" />
+            <geometry>
+                <mesh
+                    filename="file://$(find robot_arm_description)/meshes/Center_arm_bearing_guide_clamp__2__1.stl"
+                    scale="0.001 0.001 0.001" />
+            </geometry>
+        </collision>
+    </link>
     <link name="Upper_arm_left__1__1">
         <inertial>
@@ -901,5 +1073,12 @@
             <material name="silver" />
         </visual>
-        </link>
+        <collision>
+            <origin xyz="-0.00055 -0.030465 -0.251448" rpy="0 0 0" />
+            <geometry>
+                <mesh filename="file://$(find robot_arm_description)/meshes/Bearing_guide__1__1.stl"
+                    scale="0.001 0.001 0.001" />
+            </geometry>
+        </collision>
+    </link>
     <link name="Bearing_top-bottom_bushing__2__1">
         <inertial>
@@ -918,5 +1097,13 @@
             <material name="silver" />
         </visual>
-        </link>
+        <collision>
+            <origin xyz="-0.00055 -0.030465 -0.251448" rpy="0 0 0" />
+            <geometry>
+                <mesh
+                    filename="file://$(find robot_arm_description)/meshes/Bearing_top-bottom_bushing__2__1.stl"
+                    scale="0.001 0.001 0.001" />
+            </geometry>
+        </collision>
+    </link>
     <link name="Bearing_center_bushing__1__1">
         <inertial>
@@ -935,5 +1122,13 @@
             <material name="silver" />
         </visual>
-        </link>
+        <collision>
+            <origin xyz="-0.000531 -0.03046 -0.280948" rpy="0 0 0" />
+            <geometry>
+                <mesh
+                    filename="file://$(find robot_arm_description)/meshes/Bearing_center_bushing__1__1.stl"
+                    scale="0.001 0.001 0.001" />
+            </geometry>
+        </collision>
+    </link>
     <link name="Bearing_top-bottom_bushing__1__1">
         <inertial>
@@ -952,5 +1147,13 @@
             <material name="silver" />
         </visual>
-        </link>
+        <collision>
+            <origin xyz="-0.000531 -0.03046 -0.280948" rpy="0 0 0" />
+            <geometry>
+                <mesh
+                    filename="file://$(find robot_arm_description)/meshes/Bearing_top-bottom_bushing__1__1.stl"
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